Commit message: corrected inertial parameters in franka.urdf

File: src/thunder/robots/debug/franka.urdf (robot description, URDF)
Before this commit: robot panda, 13 links, 12 joints
Links:
- link panda_link0: mass 3.06 -> 0.629769
- link panda_link1: mass 2.34 -> 4.970684
- link panda_link2: mass 2.36 -> 0.646926
- link panda_link3: mass 2.38 -> 3.228604
- link panda_link4: mass 2.43 -> 3.587895
- link panda_link5: mass 3.5 -> 1.225946
- link panda_link6: mass 1.47 -> 1.666555
- link panda_link7: mass 0.45 -> 1e-10
- link panda_link8: mass 1e-10 -> 0.735522
