Commit message: bugfix origin transform urdf

File: robots/franka/franka.urdf (robot description, URDF)
Before this commit: robot panda, 13 links, 12 joints
Links:
- link panda_link7: mass 1e-10 -> None

File: src/thunder/tests/fixtures/franka/franka_symbolic.urdf (robot description, URDF)
Before this commit: robot panda, 11 links, 10 joints
Links:
- added link panda_ee, mass 1e-10
- added link panda_rightfinger, mass 0.01; collision mesh filename=package://franka_description/meshes/collision/finger.stl; visual mesh filename=package://franka_description/meshes/visual/finger.dae
Joints:
- added joint panda_ee_joint: type fixed, parent panda_link8, child panda_ee, origin xyz=0 0 0.103 rpy=0 0 -0.785398163397
- added joint panda_finger_joint2: type prismatic, parent panda_hand, child panda_rightfinger, origin xyz=0 0 0.0584 rpy=0 0 0, axis 0 -1 0, limit lower=0.0 upper=0.04 effort=20 velocity=0.2, mimic joint=panda_finger_joint1
